File: Eagle/dobbelsteen.sch (EAGLE design)
At the start: 22 parts, among them IC1 TINY24/44/84-PU

Commit message: update schematic and add fritzing
Parts:
- removed LED10, LED11, LED12, LED13, LED14, LED8, LED9: (no value), led:LED3MM
- removed S1: (no value), switch:255SB
- added R6, R7: 160, rcl:R-EU_0204/7
- added R8: 1M, rcl:R-EU_0204/7
- added TOUCH, TOUCH_GND: TPPAD1-20Y, testpad:TPPAD1-20Y
- LED1, LED2, LED3, LED4, LED5, LED6, LED7: device led:LED3MM -> led:LED5MM
- R1, R2, R3, R4, R5: value 30 -> 160; device rcl:R-EU_0309/12 -> rcl:R-EU_0204/7
Connections:
- removed net CP_A: IC1.(PCINT0/AREF/ADC0)PA0, R1.1
- removed net CP_B: IC1.(PCINT1/AIN0/ADC1)PA1, R2.1
- removed net CP_C: IC1.(PCINT2/AIN1/ADC2)PA2, R3.1
- removed net CP_D: IC1.(PCINT3/T0/ADC3)PA3, R4.1
- removed net CP_E: IC1.(PCINT4/T1/SCL/USCK/ADC4)PA4, R5.1
- new net D_CENTR: IC1.(PCINT5/OC1B/MISO/DO/ADC5)PA5, LED4.A
- new net D_DIAG1: IC1.(PCINT4/T1/SCL/USCK/ADC4)PA4, LED1.A, LED7.A
- new net D_DIAG2: IC1.(PCINT3/T0/ADC3)PA3, LED3.A, LED5.A
- new net D_HORIZ: IC1.(PCINT2/AIN1/ADC2)PA2, LED2.A, LED6.A
- new net N$7: LED7.C, R7.2
- new net N$8: IC1.(PCINT10/INT0/OC0A/CKOUT)PB2, R8.1
- new net TOUCH: IC1.(PCINT7/ICP/OC0B/ADC7)PA7, R8.2, TOUCH.TP
- net GND: now also R1.1, R2.1, R3.1, R4.1, R5.1, R6.1, R7.1, TOUCH_GND.TP; no longer S1.S
- net N$1: now also LED1.C, R1.2; no longer IC1.(PCINT8/XTAL1/CLKI)PB0, S1.P
- net N$2: now also R2.2; no longer LED1.A, LED10.C, LED9.A, R1.2
- net N$3: now also LED3.C, R3.2; no longer LED1.C, LED11.A, LED12.C, LED2.A, LED3.A, LED4.C, R2.2
- net N$4: now also LED4.C, R4.2; no longer LED10.A, LED13.A, LED14.C, LED3.C, LED4.A, LED5.A, LED6.C, LED9.C, R3.2
- net N$5: now also R5.2; no longer LED11.C, LED12.A, LED6.A, LED7.A, LED8.C, R4.2
- net N$6: now also LED6.C, R6.2; no longer LED13.C, LED14.A, LED7.C, LED8.A, R5.2
Other:
- moved on the sheet: LED1, LED2, LED3, LED4, LED5, LED6, LED7, R1, R2, R3, R4, R5
